Commit message: ros2 control toggle switching

File: description/robot.urdf.xacro (robot description, xacro)
@@ -1,4 +1,14 @@
 <?xml version="1.0"?>
 <robot xmlns:xacro="http://www.ros.org/wiki/xacro"  name="robot">
+    <xacro:arg name="use_ros2_control" default="true"/>
     <xacro:include filename="robot_core.xacro" />
+    <xacro:if value="$(arg use_ros2_control)">
+        <xacro:include filename="ros2_control.xacro" />
+    </xacro:if>
+    <xacro:unless value="$(arg use_ros2_control)">
+        <xacro:include filename="gazebo_control.xacro" />
+    </xacro:unless>
+    <!-- <xacro:include filename="lidar.xacro" /> -->
+    <xacro:include filename="camera.xacro" />
+    <!-- <xacro:include filename="depth_camera.xacro" /> -->
 </robot>

File: description/robot_core.xacro (robot description, xacro)
@@ -51,4 +51,9 @@
         </xacro:inertial_box>
     </link>
+    <gazebo reference="body">
+            <material>Gazebo/White</material>
+            <mul1>0.01</mul1>
+            <mul2>0.01</mul2>
+        </gazebo>
     <!-- LEFT FRONT WHEEL LINK-->
     <joint name="left_front_wheel_joint" type="continuous">
@@ -74,4 +79,9 @@
         </xacro:inertial_cylinder>
     </link>
+    <gazebo reference="left_front_wheel">
+            <material>Gazebo/Black</material>
+            <mul1>0.01</mul1>
+            <mul2>0.01</mul2>
+        </gazebo>
     <!-- RIGHT FRONT WHEEL LINK-->
     <joint name="right_front_wheel_joint" type="continuous">
@@ -97,4 +107,9 @@
         </xacro:inertial_cylinder>
     </link>
+    <gazebo reference="right_front_wheel">
+            <material>Gazebo/Black</material>
+            <mul1>0.01</mul1>
+            <mul2>0.01</mul2>
+        </gazebo>
     <!-- LEFT REAR WHEEL LINK-->
     <joint name="left_rear_wheel_joint" type="continuous">
@@ -120,4 +135,9 @@
         </xacro:inertial_cylinder>
     </link>
+    <gazebo reference="left_rear_wheel">
+            <material>Gazebo/Black</material>
+            <mul1>0.01</mul1>
+            <mul2>0.01</mul2>
+        </gazebo>
     <!-- RIGHT REAR WHEEL LINK-->
     <joint name="right_rear_wheel_joint" type="continuous">
@@ -143,3 +163,8 @@
         </xacro:inertial_cylinder>
     </link>
+    <gazebo reference="right_rear_wheel">
+            <material>Gazebo/Black</material>
+            <mul1>0.01</mul1>
+            <mul2>0.01</mul2>
+        </gazebo>
 </robot>
